File: Driver/MCU.kicad_sch (KiCad schematic)
At the start: 28 parts, among them IC1 STM32G474RET6, IC2 ESDA6V1L, J1 Conn_02x04_Top_Bottom, J2 ST-Link, SW1 SW_Push, SW2 SW_Push, Y2 TG2520SMN-32.0Mhz

Commit message: Update
Parts:
- SW1, SW2: footprint Button_Switch_SMD:SW_SPST_EVQPE1 -> Button_Switch_SMD:SW_Tactile_SPST_NO_Straight_CK_PTS636Sx25SMTRLFS
Changed lines of the file:
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@@
 			)
 		)
-		(property "Footprint" "Button_Switch_SMD:SW_SPST_EVQPE1"
+		(property "Footprint" "Button_Switch_SMD:SW_Tactile_SPST_NO_Straight_CK_PTS636Sx25SMTRLFS"
 			(at 127 137.16 0)
 			(effects
@@
 			)
 		)
-		(property "Footprint" "Button_Switch_SMD:SW_SPST_EVQPE1"
+		(property "Footprint" "Button_Switch_SMD:SW_Tactile_SPST_NO_Straight_CK_PTS636Sx25SMTRLFS"
 			(at 80.01 153.67 0)
 			(effects
