File: Driver/Driver.kicad_pcb (KiCad board)
At the start: 4 copper layers, 65.5 x 107 mm, 96 parts, among them IC1 STM32G474RET6, IC2 ESDA6V1L, IC3 DRV8317HREER, J1 Conn_02x04_Top_Bottom, J2 ST-Link, J5 Jack-DC, J6 Screw_Terminal_01x03, U1 LM2596S-ADJ, U2 LM2674M-5.0, U3 LD1117S33TR, Y2 TG2520SMN-32.0Mhz

Commit message: Big Change
Seperate a boards
Parts:
- J4: renamed from Encoder Knob
- J7: renamed from IMU 
- moved J1 64.1 mm to (211.3, 109.7)
- renumbered PWR to D2, PA5 to D4, Encoder to J3, Gain to JP2, Mode to JP3, Slew to JP4, RESET to SW1, USER to SW2
Connections:
- C11 pad 1: VIN_AVDD -> VDD
- C12 pad 1: VIN_AVDD -> VM
- C2 pad 1: VIN_AVDD -> VM
- C20 pad 1: VIN_AVDD -> VM
- C22 pad 1: VIN_AVDD -> VM
- C26 pad 1: VIN_AVDD -> VDD
- C3 pad 2: VIN_AVDD -> VM
- IC3 pad 20: VIN_AVDD -> VM
- IC3 pad 7: VIN_AVDD -> VDD
- IC3 pad 8: VIN_AVDD -> VM
- IC3 pad 9: VIN_AVDD -> VM
- L1 pad 2: VIN_AVDD -> VM
- RV1 pad 2: VIN_AVDD -> VM
- TP1 pad 1: VIN_AVDD -> VM
Routing:
- net VIN_AVDD: track 86.5 -> 0.00 mm, vias 81 -> 0
- net VM: track 0.00 -> 77.2 mm, vias 0 -> 72
- net /3-Phase Driver/TIM1_CH2: track 41.5 -> 0.00 mm, vias 7 -> 0
- net /External Sensor and Encoder/IMU_CS: track 37.6 -> 0.00 mm
- net /3-Phase Driver/TIM1_CH3N: track 35.0 -> 0.00 mm, vias 1 -> 0
- net /External Sensor and Encoder/IMU_SCLK: track 30.6 -> 0.00 mm, vias 2 -> 0
- net /External Sensor and Encoder/IMU_MISO: track 28.7 -> 0.00 mm, vias 1 -> 0
- net /3-Phase Driver/TIM1_CH1N: track 27.8 -> 0.00 mm, vias 2 -> 0
- net /3-Phase Driver/TIM1_CH2N: track 26.6 -> 0.00 mm, vias 3 -> 0
- net /External Sensor and Encoder/IMU_INT1: track 26.2 -> 0.00 mm
- net /3-Phase Driver/TIM1_CH1: track 26.0 -> 0.00 mm, vias 2 -> 0
- net /External Sensor and Encoder/IMU_MOSI: track 25.9 -> 0.00 mm
- net /3-Phase Driver/TIM1_CH3: track 21.0 -> 0.00 mm, vias 2 -> 0
- net CP: track 12.4 -> 0.00 mm, vias 2 -> 0
- net VDD: track 73.7 -> 69.4 mm
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- added copper zone on F.Cu, net VM
- added copper zone on In1.Cu, net VM
- removed copper zone on F.Cu, net VIN_AVDD
- removed copper zone on In1.Cu, net VIN_AVDD
