File: DRV8317-Driver/Driver-DRV8317/PSU.kicad_sch (KiCad schematic)
At the start: 25 parts, among them J5 Jack-DC, U1 LM2596S-ADJ, U2 LM2674M-5.0, U3 LD1117S33TR

Commit message: kncoadsnofijasndvoi
Parts:
- added D5: Red LED, LED_SMD:LED_0805_2012Metric, symbol Device:LED
- added R34, R35: 3.6, Resistor_SMD:R_0805_2012Metric, symbol Device:R
Connections:
- net +3.3V: now also R34.1
- net GND: now also D5.1 (K)
- new net: D5.2 (A), R35.2
- new net: R34.2, R35.1
Other:
- moved on the sheet: C1, C2, C3, D1, L1, R3, RV1, TP1, TP2, U1
