File: IMU/IMU.kicad_sch (KiCad schematic)
At the start: 7 parts, among them IC1 ICM-42688-P, J2 IMU

Commit message: Up
Parts:
- C1: value 0.01uF X7R -> 10nF X7R
Changed lines of the file:
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@@
 			)
 		)
-		(property "Value" "0.01uF X7R"
+		(property "Value" "10nF X7R"
 			(at 127 139.7 90)
 			(effects
