File: MCU/ConnAndSensor.kicad_sch (KiCad schematic)
At the start: 20 parts, among them J3 Encoder1, J4 Encoder2, J5 Conn_02x13_Odd_Even, J7 IMU

Commit message: kncoadsnofijasndvoi
Parts:
- R34, R35: footprint Resistor_SMD:R_0603_1608Metric -> Resistor_SMD:R_0805_2012Metric
Changed lines of the file:
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@@
 			)
 		)
-		(property "Footprint" "Resistor_SMD:R_0603_1608Metric"
+		(property "Footprint" "Resistor_SMD:R_0805_2012Metric"
 			(at 233.68 113.538 90)
 			(effects
@@
 			)
 		)
-		(property "Footprint" "Resistor_SMD:R_0603_1608Metric"
+		(property "Footprint" "Resistor_SMD:R_0805_2012Metric"
 			(at 223.52 113.538 90)
 			(effects

Commit message: fix all via to 0.45/0.3 mm
Parts:
- TP1, TP2, TP3: footprint Connector_Pin:Pin_D0.7mm_L6.5mm_W1.8mm_FlatFork -> TestPoint:TestPoint_Loop_D1.80mm_Drill1.0mm_Beaded
Changed lines of the file:
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@@
 			)
 		)
-		(property "Footprint" "Connector_Pin:Pin_D0.7mm_L6.5mm_W1.8mm_FlatFork"
+		(property "Footprint" "TestPoint:TestPoint_Loop_D1.80mm_Drill1.0mm_Beaded"
 			(at 172.72 110.49 0)
 			(effects
@@
 			)
 		)
-		(property "Footprint" "Connector_Pin:Pin_D0.7mm_L6.5mm_W1.8mm_FlatFork"
+		(property "Footprint" "TestPoint:TestPoint_Loop_D1.80mm_Drill1.0mm_Beaded"
 			(at 172.72 118.11 0)
 			(effects
@@
 			)
 		)
-		(property "Footprint" "Connector_Pin:Pin_D0.7mm_L6.5mm_W1.8mm_FlatFork"
+		(property "Footprint" "TestPoint:TestPoint_Loop_D1.80mm_Drill1.0mm_Beaded"
 			(at 172.72 104.14 0)
 			(effects
