File: MCU/MCUs.kicad_sch (KiCad schematic)
At the start: 28 parts, among them IC1 STM32G474RET6, IC2 ESDA6V1L, J1 Conn_02x04_Top_Bottom, J2 ST-Link, SW1 SW_Push, SW2 SW_Push, Y2 TG2520SMN-32.0Mhz

Commit message: kncoadsnofijasndvoi
Parts:
- R30, R31: footprint Resistor_SMD:R_0603_1608Metric -> Resistor_SMD:R_0805_2012Metric
Changed lines of the file:
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@@
 			)
 		)
-		(property "Footprint" "Resistor_SMD:R_0603_1608Metric"
+		(property "Footprint" "Resistor_SMD:R_0805_2012Metric"
 			(at 189.23 124.968 90)
 			(effects
@@
 			)
 		)
-		(property "Footprint" "Resistor_SMD:R_0603_1608Metric"
+		(property "Footprint" "Resistor_SMD:R_0805_2012Metric"
 			(at 199.39 124.968 90)
 			(effects

Commit message: fix all via to 0.45/0.3 mm
Connections:
- net TIM1_CH1: now also J1.5 (Pin_5); no longer J1.3 (Pin_3)
- net TIM1_CH1N: no longer J1.4 (Pin_4)
- net TIM1_CH2: now also J1.2 (Pin_2); no longer J1.1 (Pin_1)
- net TIM1_CH2N: now also J1.4 (Pin_4); no longer J1.2 (Pin_2)
- net TIM1_CH3: now also J1.1 (Pin_1); no longer J1.5 (Pin_5)
- net TIM1_CH3N: now also J1.3 (Pin_3); no longer J1.6 (Pin_6)
Changed lines of the file:
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@@
 	(hierarchical_label "TIM1_CH1"
 		(shape output)
+		(at 205.74 144.78 0)
+		(effects
+			(font
+				(size 1.27 1.27)
+			)
+			(justify left)
+		)
+	)
+	(hierarchical_label "TIM1_CH2N"
+		(shape output)
+		(at 193.04 152.4 180)
+		(effects
+			(font
+				(size 1.27 1.27)
+			)
+			(justify right)
+		)
+	)
+	(hierarchical_label "TIM1_CH1"
+		(shape output)
 		(at 261.62 66.04 0)
 		(effects
@@
 		)
 	)
+	(hierarchical_label "TIM1_CH2"
+		(shape output)
+		(at 261.62 60.96 0)
+		(effects
+			(font
+				(size 1.27 1.27)
+			)
+			(justify left)
+		)
+	)
+	(hierarchical_label "Button"
+		(shape input)
+		(at 231.14 27.94 90)
+		(effects
+			(font
+				(size 1.27 1.27)
+			)
+			(justify left)
+		)
+	)
+	(hierarchical_label "IMU_INT1"
+		(shape input)
+		(at 261.62 86.36 0)
+		(effects
+			(font
+				(size 1.27 1.27)
+			)
+			(justify left)
+		)
+	)
+	(hierarchical_label "IMU_INT2"
+		(shape input)
+		(at 261.62 88.9 0)
+		(effects
+			(font
+				(size 1.27 1.27)
+			)
+			(justify left)
+		)
+	)
+	(hierarchical_label "Encoder2 B"
+		(shape input)
+		(at 226.06 27.94 90)
+		(effects
+			(font
+				(size 1.27 1.27)
+			)
+			(justify left)
+		)
+	)
+	(hierarchical_label "Encoder1 A"
+		(shape input)
+		(at 223.52 106.68 270)
+		(effects
+			(font
+				(size 1.27 1.27)
+			)
+			(justify right)
+		)
+	)
+	(hierarchical_label "NFAULT"
+		(shape input)
+		(at 205.74 149.86 0)
+		(effects
+			(font
+				(size 1.27 1.27)
+			)
+			(justify left)
+		)
+	)
+	(hierarchical_label "TIM1_CH3N"
+		(shape output)
+		(at 193.04 149.86 180)
+		(effects
+			(font
+				(size 1.27 1.27)
+			)
+			(justify right)
+		)
+	)
+	(hierarchical_label "IMU_MISO"
+		(shape input)
+		(at 261.62 81.28 0)
+		(effects
+			(font
+				(size 1.27 1.27)
+			)
+			(justify left)
+		)
+	)
+	(hierarchical_label "Vcurrfdbk_B"
+		(shape input)
+		(at 205.74 71.12 180)
+		(effects
+			(font
+				(size 1.27 1.27)
+			)
+			(justify right)
+		)
+	)
+	(hierarchical_label "TIM1_CH3"
+		(shape output)
+		(at 261.62 71.12 0)
+		(effects
+			(font
+				(size 1.27 1.27)
+			)
+			(justify left)
+		)
+	)
+	(hierarchical_label "Encoder2 A"
+		(shape input)
+		(at 228.6 27.94 90)
+		(effects
+			(font
+				(size 1.27 1.27)
+			)
+			(justify left)
+		)
+	)
+	(hierarchical_label "TIM1_CH3N"
+		(shape output)
+		(at 261.62 68.58 0)
+		(effects
+			(font
+				(size 1.27 1.27)
+			)
+			(justify left)
+		)
+	)
+	(hierarchical_label "Vcurrfdbk_C"
+		(shape input)
+		(at 205.74 73.66 180)
+		(effects
+			(font
+				(size 1.27 1.27)
+			)
+			(justify right)
+		)
+	)
 	(hierarchical_label "TIM1_CH1N"
 		(shape output)
-		(at 193.04 152.4 180)
-		(effects
-			(font
-				(size 1.27 1.27)
-			)
-			(justify right)
+		(at 261.62 63.5 0)
+		(effects
+			(font
+				(size 1.27 1.27)
+			)
+			(justify left)
+		)
+	)
+	(hierarchical_label "IMU_SCLK"
+		(shape output)
+		(at 261.62 83.82 0)
+		(effects
+			(font
+				(size 1.27 1.27)
+			)
+			(justify left)
+		)
+	)
+	(hierarchical_label "IMU_CS"
+		(shape output)
+		(at 261.62 76.2 0)
+		(effects
+			(font
+				(size 1.27 1.27)
+			)
+			(justify left)
 		)
 	)
 	(hierarchical_label "TIM1_CH2"
 		(shape output)
-		(at 261.62 60.96 0)
-		(effects
-			(font
-				(size 1.27 1.27)
-			)
-			(justify left)
-		)
-	)
-	(hierarchical_label "Button"
-		(shape input)
-		(at 231.14 27.94 90)
+		(at 193.04 147.32 180)
+		(effects
+			(font
+				(size 1.27 1.27)
+			)
+			(justify right)
+		)
+	)
+	(hierarchical_label "NSLEEP"
+		(shape output)
+		(at 261.62 73.66 0)
+		(effects
+			(font
+				(size 1.27 1.27)
+			)
+			(justify left)
+		)
+	)
+	(hierarchical_label "IMU_MOSI"
+		(shape output)
+		(at 261.62 78.74 0)
 		(effects
 			(font
@@
 	(hierarchical_label "TIM1_CH2N"
 		(shape output)
-		(at 193.04 147.32 180)
-		(effects
-			(font
-				(size 1.27 1.27)
-			)
-			(justify right)
-		)
-	)
-	(hierarchical_label "IMU_INT1"
-		(shape input)
-		(at 261.62 86.36 0)
-		(effects
-			(font
-				(size 1.27 1.27)
-			)
-			(justify left)
-		)
-	)
-	(hierarchical_label "IMU_INT2"
-		(shape input)
-		(at 261.62 88.9 0)
-		(effects
-			(font
-				(size 1.27 1.27)
-			)
-			(justify left)
-		)
-	)
-	(hierarchical_label "Encoder2 B"
-		(shape input)
-		(at 226.06 27.94 90)
-		(effects
-			(font
-				(size 1.27 1.27)
-			)
-			(justify left)
-		)
-	)
-	(hierarchical_label "Encoder1 A"
-		(shape input)
-		(at 223.52 106.68 270)
-		(effects
-			(font
-				(size 1.27 1.27)
-			)
-			(justify right)
+		(at 261.62 58.42 0)
+		(effects
+			(font
+				(size 1.27 1.27)
+			)
+			(justify left)
 		)
 	)
 	(hierarchical_label "NFAULT"
 		(shape input)
-		(at 205.74 149.86 0)
-		(effects
-			(font
-				(size 1.27 1.27)
-			)
-			(justify left)
-		)
-	)
-	(hierarchical_label "IMU_MISO"
-		(shape input)
-		(at 261.62 81.28 0)
-		(effects
-			(font
-				(size 1.27 1.27)
-			)
-			(justify left)
-		)
-	)
-	(hierarchical_label "Vcurrfdbk_B"
-		(shape input)
-		(at 205.74 71.12 180)
-		(effects
-			(font
-				(size 1.27 1.27)
-			)
-			(justify right)
+		(at 261.62 55.88 0)
+		(effects
+			(font
+				(size 1.27 1.27)
+			)
+			(justify left)
 		)
 	)
 	(hierarchical_label "TIM1_CH3"
 		(shape output)
-		(at 261.62 71.12 0)
-		(effects
-			(font
-				(size 1.27 1.27)
-			)
-			(justify left)
-		)
-	)
-	(hierarchical_label "Encoder2 A"
-		(shape input)
-		(at 228.6 27.94 90)
-		(effects
-			(font
-				(size 1.27 1.27)
-			)
-			(justify left)
-		)
-	)
-	(hierarchical_label "TIM1_CH3N"
-		(shape output)
-		(at 261.62 68.58 0)
-		(effects
-			(font
-				(size 1.27 1.27)
-			)
-			(justify left)
-		)
-	)
-	(hierarchical_label "TIM1_CH1"
-		(shape output)
-		(at 193.04 149.86 180)
-		(effects
-			(font
-				(size 1.27 1.27)
-			)
-			(justify right)
-		)
-	)
-	(hierarchical_label "Vcurrfdbk_C"
-		(shape input)
-		(at 205.74 73.66 180)
-		(effects
-			(font
-				(size 1.27 1.27)
-			)
-			(justify right)
-		)
-	)
-	(hierarchical_label "TIM1_CH1N"
-		(shape output)
-		(at 261.62 63.5 0)
-		(effects
-			(font
-				(size 1.27 1.27)
-			)
-			(justify left)
-		)
-	)
-	(hierarchical_label "IMU_SCLK"
-		(shape output)
-		(at 261.62 83.82 0)
-		(effects
-			(font
-				(size 1.27 1.27)
-			)
-			(justify left)
-		)
-	)
-	(hierarchical_label "IMU_CS"
-		(shape output)
-		(at 261.62 76.2 0)
-		(effects
-			(font
-				(size 1.27 1.27)
-			)
-			(justify left)
-		)
-	)
-	(hierarchical_label "TIM1_CH2"
-		(shape output)
 		(at 193.04 144.78 180)
 		(effects
@@
 		)
 	)
-	(hierarchical_label "TIM1_CH3"
-		(shape output)
-		(at 205.74 144.78 0)
-		(effects
-			(font
-				(size 1.27 1.27)
-			)
-			(justify left)
-		)
-	)
-	(hierarchical_label "NSLEEP"
-		(shape output)
-		(at 261.62 73.66 0)
-		(effects
-			(font
-				(size 1.27 1.27)
-			)
-			(justify left)
-		)
-	)
-	(hierarchical_label "IMU_MOSI"
-		(shape output)
-		(at 261.62 78.74 0)
-		(effects
-			(font
-				(size 1.27 1.27)
-			)
-			(justify left)
-		)
-	)
-	(hierarchical_label "TIM1_CH2N"
-		(shape output)
-		(at 261.62 58.42 0)
-		(effects
-			(font
-				(size 1.27 1.27)
-			)
-			(justify left)
-		)
-	)
-	(hierarchical_label "NFAULT"
-		(shape input)
-		(at 261.62 55.88 0)
-		(effects
-			(font
-				(size 1.27 1.27)
-			)
-			(justify left)
-		)
-	)
-	(hierarchical_label "TIM1_CH3N"
-		(shape output)
-		(at 205.74 147.32 0)
-		(effects
-			(font
-				(size 1.27 1.27)
-			)
-			(justify left)
-		)
-	)
